Commit message: 适配rtk_gps

File: lio-sam-workspace/src/LIO-SAM/launch/include/config/robot.urdf.xacro (robot description, xacro)
@@ -15,21 +15,21 @@
     <origin xyz="0 0 0" rpy="0 0 0" />
   </joint>
-  <link name="imu_link"> </link>
+  <!-- <link name="imu_link"> </link>
   <joint name="imu_joint" type="fixed">
     <parent link="chassis_link" />
     <child link="imu_link" />
     <origin xyz="0 0 0" rpy="0 0 0" />
-  </joint>
-  <link name="navsat_link"> </link>
+  </joint> -->
+  <!-- <link name="navsat_link"> </link>
   <joint name="navsat_joint" type="fixed">
     <parent link="chassis_link" />
     <child link="navsat_link" />
     <origin xyz="0 0 0" rpy="0 0 0" />
-  </joint>
-  <!-- <link name="rtk_link"> </link>
+  </joint> -->
+  <link name="rtk_link"> </link>
   <joint name="rtk_joint" type="fixed">
     <parent link="base_link" />
     <child link="rtk_link" />
-    <origin xyz="0 0 0" rpy="0 0 0" />
-  </joint> -->
+    <origin xyz="-0.5 -0.5 -1" rpy="0 0 0" />
+  </joint>
 </robot>
